File: pcb/kb-pcb.kicad_pcb (KiCad board)
At the start: 2 copper layers, 269 x 101.4 mm, 151 parts, among them U1 TEENSY2.0

Commit message: upgrade to Kicad 5 footprints
In doing so, I've updated the diodes to be N4148 diodes from the
official modules. Since those have slightly different footprints from
the original ones I used, I've modified the PCB layout accordingly.

I lost track of the original Teensy 2.0 footprint I created, so I'm
using a modified version of XenGi's footprint as well.
Parts:
- D1, D10, D11, D12, D13, D14, D15, D16, D17, D18, D19, D2, D20, D21, D22, D23, D24, D25, D26, D27, D28, D29, D3, D30, D31, D32, D33, D34, D35, D36, D37, D38, D39, D4, D40, D41, D42, D43, D44, D45, D46, D47, D48, D49, D5, D50, D51, D52, D53, D54, D55, D56, D57, D58, D59, D6, D60, D61, D62, D63, D64, D65, D66, D67, D68, D7, D8, D9: footprint modded_keyboard_components:diode -> Diode_THT:D_DO-35_SOD27_P7.62mm_Horizontal
- U1: footprint modded_keyboard_components:TEENSY_2.0 -> teensy:Teensy2.0; moved to F.Cu
- moved D63 8.91 mm to (320.9, 146.1), turned to 180 degrees
- moved D38 8.90 mm to (351.8, 108.5), turned to 180 degrees
- moved D39 8.89 mm to (370.8, 108.2), turned to 180 degrees
- moved D40 8.89 mm to (389.9, 108.2), turned to 180 degrees
- moved D41 8.89 mm to (408.9, 108.2), turned to 180 degrees
- moved D10 8.89 mm to (351.8, 69.8), turned to 180 degrees
- moved D24 8.89 mm to (351.8, 88.9), turned to 180 degrees
- moved D52 8.89 mm to (351.8, 127.0), turned to 180 degrees
- moved D1 8.89 mm to (180.3, 69.8), turned to 180 degrees
- moved D15 8.89 mm to (180.3, 88.9), turned to 180 degrees
- moved D18 8.89 mm to (237.5, 88.9), turned to 180 degrees
- moved D19 8.89 mm to (256.5, 88.9), turned to 180 degrees
- moved D29 8.89 mm to (180.3, 108.0), turned to 180 degrees
- moved D32 8.89 mm to (237.5, 108.0), turned to 180 degrees
- moved D33 8.89 mm to (256.5, 108.0), turned to 180 degrees
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Connections:
- D15 pad 1: Net-(D15-Pad1) -> Net-(D1-Pad1)
- D15 pad 2: Net-(D1-Pad2) -> Net-(D15-Pad2)
- D2 pad 1: Net-(D2-Pad1) -> Net-(D16-Pad1)
- D2 pad 2: Net-(D16-Pad2) -> Net-(D2-Pad2)
- D24 pad 1: Net-(D24-Pad1) -> Net-(D10-Pad1)
- D24 pad 2: Net-(D10-Pad2) -> Net-(D24-Pad2)
- D25 pad 1: Net-(D25-Pad1) -> Net-(D11-Pad1)
- D25 pad 2: Net-(D11-Pad2) -> Net-(D25-Pad2)
- D26 pad 1: Net-(D26-Pad1) -> Net-(D12-Pad1)
- D26 pad 2: Net-(D12-Pad2) -> Net-(D26-Pad2)
- D27 pad 1: Net-(D27-Pad1) -> Net-(D13-Pad1)
- D27 pad 2: Net-(D13-Pad2) -> Net-(D27-Pad2)
- D28 pad 1: Net-(D28-Pad1) -> Net-(D14-Pad1)
- D28 pad 2: Net-(D14-Pad2) -> Net-(D28-Pad2)
- D29 pad 1: Net-(D29-Pad1) -> Net-(D1-Pad1)
- D29 pad 2: Net-(D1-Pad2) -> Net-(D29-Pad2)
- D3 pad 1: Net-(D3-Pad1) -> Net-(D17-Pad1)
- D3 pad 2: Net-(D17-Pad2) -> Net-(D3-Pad2)
- D30 pad 1: Net-(D30-Pad1) -> Net-(D16-Pad1)
- D30 pad 2: Net-(D16-Pad2) -> Net-(D30-Pad2)
- D31 pad 1: Net-(D31-Pad1) -> Net-(D17-Pad1)
- D31 pad 2: Net-(D17-Pad2) -> Net-(D31-Pad2)
- D32 pad 1: Net-(D32-Pad1) -> Net-(D18-Pad1)
- D32 pad 2: Net-(D18-Pad2) -> Net-(D32-Pad2)
- D33 pad 1: Net-(D33-Pad1) -> Net-(D19-Pad1)
- D33 pad 2: Net-(D19-Pad2) -> Net-(D33-Pad2)
- D34 pad 1: Net-(D34-Pad1) -> Net-(D20-Pad1)
- D34 pad 2: Net-(D20-Pad2) -> Net-(D34-Pad2)
- D35 pad 1: Net-(D35-Pad1) -> Net-(D21-Pad1)
- D35 pad 2: Net-(D21-Pad2) -> Net-(D35-Pad2)
- D36 pad 1: Net-(D36-Pad1) -> Net-(D22-Pad1)
- D36 pad 2: Net-(D22-Pad2) -> Net-(D36-Pad2)
- D37 pad 1: Net-(D37-Pad1) -> Net-(D23-Pad1)
- D37 pad 2: Net-(D23-Pad2) -> Net-(D37-Pad2)
- D38 pad 1: Net-(D38-Pad1) -> Net-(D10-Pad1)
- D38 pad 2: Net-(D10-Pad2) -> Net-(D38-Pad2)
- D39 pad 1: Net-(D39-Pad1) -> Net-(D11-Pad1)
- D39 pad 2: Net-(D11-Pad2) -> Net-(D39-Pad2)
- D4 pad 1: Net-(D4-Pad1) -> Net-(D18-Pad1)
- D4 pad 2: Net-(D18-Pad2) -> Net-(D4-Pad2)
- D40 pad 1: Net-(D40-Pad1) -> Net-(D12-Pad1)
- D40 pad 2: Net-(D12-Pad2) -> Net-(D40-Pad2)
- D41 pad 1: Net-(D41-Pad1) -> Net-(D13-Pad1)
- D41 pad 2: Net-(D13-Pad2) -> Net-(D41-Pad2)
- D42 pad 1: Net-(D42-Pad1) -> Net-(D14-Pad1)
- D42 pad 2: Net-(D14-Pad2) -> Net-(D42-Pad2)
- D43 pad 1: Net-(D43-Pad1) -> Net-(D1-Pad1)
- D43 pad 2: Net-(D1-Pad2) -> Net-(D43-Pad2)
- D44 pad 1: Net-(D44-Pad1) -> Net-(D16-Pad1)
- D44 pad 2: Net-(D16-Pad2) -> Net-(D44-Pad2)
- D45 pad 1: Net-(D45-Pad1) -> Net-(D17-Pad1)
- D45 pad 2: Net-(D17-Pad2) -> Net-(D45-Pad2)
- D46 pad 1: Net-(D46-Pad1) -> Net-(D18-Pad1)
- D46 pad 2: Net-(D18-Pad2) -> Net-(D46-Pad2)
- D47 pad 1: Net-(D47-Pad1) -> Net-(D19-Pad1)
- D47 pad 2: Net-(D19-Pad2) -> Net-(D47-Pad2)
- D48 pad 1: Net-(D48-Pad1) -> Net-(D20-Pad1)
- D48 pad 2: Net-(D20-Pad2) -> Net-(D48-Pad2)
- D49 pad 1: Net-(D49-Pad1) -> Net-(D21-Pad1)
- D49 pad 2: Net-(D21-Pad2) -> Net-(D49-Pad2)
- D5 pad 1: Net-(D5-Pad1) -> Net-(D19-Pad1)
- D5 pad 2: Net-(D19-Pad2) -> Net-(D5-Pad2)
- D50 pad 1: Net-(D50-Pad1) -> Net-(D22-Pad1)
- D50 pad 2: Net-(D22-Pad2) -> Net-(D50-Pad2)
- D51 pad 1: Net-(D51-Pad1) -> Net-(D23-Pad1)
- D51 pad 2: Net-(D23-Pad2) -> Net-(D51-Pad2)
- D52 pad 1: Net-(D52-Pad1) -> Net-(D10-Pad1)
- D52 pad 2: Net-(D10-Pad2) -> Net-(D52-Pad2)
- D53 pad 1: Net-(D53-Pad1) -> Net-(D11-Pad1)
- D53 pad 2: Net-(D11-Pad2) -> Net-(D53-Pad2)
- D54 pad 1: Net-(D54-Pad1) -> Net-(D12-Pad1)
- D54 pad 2: Net-(D12-Pad2) -> Net-(D54-Pad2)
- D55 pad 1: Net-(D55-Pad1) -> Net-(D13-Pad1)
- D55 pad 2: Net-(D13-Pad2) -> Net-(D55-Pad2)
- D56 pad 1: Net-(D56-Pad1) -> Net-(D14-Pad1)
- D56 pad 2: Net-(D14-Pad2) -> Net-(D56-Pad2)
- D57 pad 1: Net-(D57-Pad1) -> Net-(D1-Pad1)
- D57 pad 2: Net-(D1-Pad2) -> Net-(D57-Pad2)
- D58 pad 1: Net-(D58-Pad1) -> Net-(D16-Pad1)
- D58 pad 2: Net-(D16-Pad2) -> Net-(D58-Pad2)
- D59 pad 1: Net-(D59-Pad1) -> Net-(D17-Pad1)
- D59 pad 2: Net-(D17-Pad2) -> Net-(D59-Pad2)
- D6 pad 1: Net-(D6-Pad1) -> Net-(D20-Pad1)
- D6 pad 2: Net-(D20-Pad2) -> Net-(D6-Pad2)
- D60 pad 1: Net-(D60-Pad1) -> Net-(D18-Pad1)
- D60 pad 2: Net-(D18-Pad2) -> Net-(D60-Pad2)
- D61 pad 1: Net-(D61-Pad1) -> Net-(D19-Pad1)
- D61 pad 2: Net-(D19-Pad2) -> Net-(D61-Pad2)
- D62 pad 1: Net-(D62-Pad1) -> Net-(D21-Pad1)
- D62 pad 2: Net-(D21-Pad2) -> Net-(D62-Pad2)
- D63 pad 1: Net-(D63-Pad1) -> Net-(D22-Pad1)
- D63 pad 2: Net-(D22-Pad2) -> Net-(D63-Pad2)
- D64 pad 1: Net-(D64-Pad1) -> Net-(D10-Pad1)
- D64 pad 2: Net-(D10-Pad2) -> Net-(D64-Pad2)
- D65 pad 1: Net-(D65-Pad1) -> Net-(D11-Pad1)
- D65 pad 2: Net-(D11-Pad2) -> Net-(D65-Pad2)
- D66 pad 1: Net-(D66-Pad1) -> Net-(D12-Pad1)
- D66 pad 2: Net-(D12-Pad2) -> Net-(D66-Pad2)
- D67 pad 1: Net-(D67-Pad1) -> Net-(D13-Pad1)
- D67 pad 2: Net-(D13-Pad2) -> Net-(D67-Pad2)
- D68 pad 1: Net-(D68-Pad1) -> Net-(D14-Pad1)
- D68 pad 2: Net-(D14-Pad2) -> Net-(D68-Pad2)
- D7 pad 1: Net-(D7-Pad1) -> Net-(D21-Pad1)
- D7 pad 2: Net-(D21-Pad2) -> Net-(D7-Pad2)
- D8 pad 1: Net-(D8-Pad1) -> Net-(D22-Pad1)
- D8 pad 2: Net-(D22-Pad2) -> Net-(D8-Pad2)
- D9 pad 1: Net-(D9-Pad1) -> Net-(D23-Pad1)
- D9 pad 2: Net-(D23-Pad2) -> Net-(D9-Pad2)
- R1 pad 1: Net-(D1-Pad2) -> Net-(D1-Pad1)
- R10 pad 1: Net-(D10-Pad2) -> Net-(D10-Pad1)
- R11 pad 1: Net-(D11-Pad2) -> Net-(D11-Pad1)
- R12 pad 1: Net-(D12-Pad2) -> Net-(D12-Pad1)
- R13 pad 1: Net-(D13-Pad2) -> Net-(D13-Pad1)
- R14 pad 1: Net-(D14-Pad2) -> Net-(D14-Pad1)
- R2 pad 1: Net-(D16-Pad2) -> Net-(D16-Pad1)
- R3 pad 1: Net-(D17-Pad2) -> Net-(D17-Pad1)
- R4 pad 1: Net-(D18-Pad2) -> Net-(D18-Pad1)
- R5 pad 1: Net-(D19-Pad2) -> Net-(D19-Pad1)
- R6 pad 1: Net-(D20-Pad2) -> Net-(D20-Pad1)
- R7 pad 1: Net-(D21-Pad2) -> Net-(D21-Pad1)
- R8 pad 1: Net-(D22-Pad2) -> Net-(D22-Pad1)
- R9 pad 1: Net-(D23-Pad2) -> Net-(D23-Pad1)
- S1 pad 1: Net-(D1-Pad1) -> Net-(D1-Pad2)
- S10 pad 1: Net-(D10-Pad1) -> Net-(D10-Pad2)
- S11 pad 1: Net-(D11-Pad1) -> Net-(D11-Pad2)
- S12 pad 1: Net-(D12-Pad1) -> Net-(D12-Pad2)
- S13 pad 1: Net-(D13-Pad1) -> Net-(D13-Pad2)
- S14 pad 1: Net-(D14-Pad1) -> Net-(D14-Pad2)
- S15 pad 1: Net-(D15-Pad1) -> Net-(D15-Pad2)
- S16 pad 1: Net-(D16-Pad1) -> Net-(D16-Pad2)
- S17 pad 1: Net-(D17-Pad1) -> Net-(D17-Pad2)
- S18 pad 1: Net-(D18-Pad1) -> Net-(D18-Pad2)
- S19 pad 1: Net-(D19-Pad1) -> Net-(D19-Pad2)
- S2 pad 1: Net-(D2-Pad1) -> Net-(D2-Pad2)
- S20 pad 1: Net-(D20-Pad1) -> Net-(D20-Pad2)
- S21 pad 1: Net-(D21-Pad1) -> Net-(D21-Pad2)
- S22 pad 1: Net-(D22-Pad1) -> Net-(D22-Pad2)
- S23 pad 1: Net-(D23-Pad1) -> Net-(D23-Pad2)
- S24 pad 1: Net-(D24-Pad1) -> Net-(D24-Pad2)
- S25 pad 1: Net-(D25-Pad1) -> Net-(D25-Pad2)
- S26 pad 1: Net-(D26-Pad1) -> Net-(D26-Pad2)
- S27 pad 1: Net-(D27-Pad1) -> Net-(D27-Pad2)
- S28 pad 1: Net-(D28-Pad1) -> Net-(D28-Pad2)
- S29 pad 1: Net-(D29-Pad1) -> Net-(D29-Pad2)
- S3 pad 1: Net-(D3-Pad1) -> Net-(D3-Pad2)
- S30 pad 1: Net-(D30-Pad1) -> Net-(D30-Pad2)
- S31 pad 1: Net-(D31-Pad1) -> Net-(D31-Pad2)
- S32 pad 1: Net-(D32-Pad1) -> Net-(D32-Pad2)
- S33 pad 1: Net-(D33-Pad1) -> Net-(D33-Pad2)
- S34 pad 1: Net-(D34-Pad1) -> Net-(D34-Pad2)
- S35 pad 1: Net-(D35-Pad1) -> Net-(D35-Pad2)
- S36 pad 1: Net-(D36-Pad1) -> Net-(D36-Pad2)
- S37 pad 1: Net-(D37-Pad1) -> Net-(D37-Pad2)
- S38 pad 1: Net-(D38-Pad1) -> Net-(D38-Pad2)
- S39 pad 1: Net-(D39-Pad1) -> Net-(D39-Pad2)
- S4 pad 1: Net-(D4-Pad1) -> Net-(D4-Pad2)
- S40 pad 1: Net-(D40-Pad1) -> Net-(D40-Pad2)
- S41 pad 1: Net-(D41-Pad1) -> Net-(D41-Pad2)
- S42 pad 1: Net-(D42-Pad1) -> Net-(D42-Pad2)
- S43 pad 1: Net-(D43-Pad1) -> Net-(D43-Pad2)
- S44 pad 1: Net-(D44-Pad1) -> Net-(D44-Pad2)
- S45 pad 1: Net-(D45-Pad1) -> Net-(D45-Pad2)
- S46 pad 1: Net-(D46-Pad1) -> Net-(D46-Pad2)
- S47 pad 1: Net-(D47-Pad1) -> Net-(D47-Pad2)
- S48 pad 1: Net-(D48-Pad1) -> Net-(D48-Pad2)
- S49 pad 1: Net-(D49-Pad1) -> Net-(D49-Pad2)
- S5 pad 1: Net-(D5-Pad1) -> Net-(D5-Pad2)
- S50 pad 1: Net-(D50-Pad1) -> Net-(D50-Pad2)
- S51 pad 1: Net-(D51-Pad1) -> Net-(D51-Pad2)
- S52 pad 1: Net-(D52-Pad1) -> Net-(D52-Pad2)
- S53 pad 1: Net-(D53-Pad1) -> Net-(D53-Pad2)
- S54 pad 1: Net-(D54-Pad1) -> Net-(D54-Pad2)
- S55 pad 1: Net-(D55-Pad1) -> Net-(D55-Pad2)
- S56 pad 1: Net-(D56-Pad1) -> Net-(D56-Pad2)
- S57 pad 1: Net-(D57-Pad1) -> Net-(D57-Pad2)
- S58 pad 1: Net-(D58-Pad1) -> Net-(D58-Pad2)
- S59 pad 1: Net-(D59-Pad1) -> Net-(D59-Pad2)
- S6 pad 1: Net-(D6-Pad1) -> Net-(D6-Pad2)
- S60 pad 1: Net-(D60-Pad1) -> Net-(D60-Pad2)
- S61 pad 1: Net-(D61-Pad1) -> Net-(D61-Pad2)
- S62 pad 1: Net-(D62-Pad1) -> Net-(D62-Pad2)
- S63 pad 1: Net-(D63-Pad1) -> Net-(D63-Pad2)
- S64 pad 1: Net-(D64-Pad1) -> Net-(D64-Pad2)
- S65 pad 1: Net-(D65-Pad1) -> Net-(D65-Pad2)
- S66 pad 1: Net-(D66-Pad1) -> Net-(D66-Pad2)
- S67 pad 1: Net-(D67-Pad1) -> Net-(D67-Pad2)
- S68 pad 1: Net-(D68-Pad1) -> Net-(D68-Pad2)
- S7 pad 1: Net-(D7-Pad1) -> Net-(D7-Pad2)
- S8 pad 1: Net-(D8-Pad1) -> Net-(D8-Pad2)
- S9 pad 1: Net-(D9-Pad1) -> Net-(D9-Pad2)
- U1 pad 2: Net-(D14-Pad2) -> Net-(D14-Pad1)
- U1 pad 20: Net-(D10-Pad2) -> Net-(D10-Pad1)
- U1 pad 21: Net-(D23-Pad2) -> Net-(D23-Pad1)
- U1 pad 22: Net-(D22-Pad2) -> Net-(D22-Pad1)
- U1 pad 23: Net-(D1-Pad2) -> Net-(D1-Pad1)
- U1 pad 24: Net-(D16-Pad2) -> Net-(D16-Pad1)
- U1 pad 25: Net-(D17-Pad2) -> Net-(D17-Pad1)
- U1 pad 26: Net-(D18-Pad2) -> Net-(D18-Pad1)
- U1 pad 27: Net-(D19-Pad2) -> Net-(D19-Pad1)
- U1 pad 28: Net-(D20-Pad2) -> Net-(D20-Pad1)
- U1 pad 3: Net-(D13-Pad2) -> Net-(D13-Pad1)
- U1 pad 4: Net-(D12-Pad2) -> Net-(D12-Pad1)
- U1 pad 5: Net-(D11-Pad2) -> Net-(D11-Pad1)
- U1 pad 6: Net-(D21-Pad2) -> Net-(D21-Pad1)
Routing:
- net Net-(D14-Pad2): track 461.7 -> 4.34 mm, vias 1 -> 0
- net Net-(D14-Pad1): track 4.86 -> 461.0 mm, vias 0 -> 1
- net Net-(D13-Pad1): track 4.86 -> 430.0 mm, vias 0 -> 1
- net Net-(D13-Pad2): track 427.8 -> 4.34 mm, vias 1 -> 0
- net Net-(D12-Pad1): track 4.86 -> 404.1 mm, vias 0 -> 1
- net Net-(D12-Pad2): track 401.9 -> 4.34 mm, vias 1 -> 0
- net Net-(D11-Pad1): track 4.86 -> 379.3 mm, vias 0 -> 2
- net Net-(D11-Pad2): track 377.2 -> 4.34 mm, vias 2 -> 0
- net Net-(D21-Pad1): track 4.86 -> 282.1 mm, vias 0 -> 6
- net Net-(D21-Pad2): track 279.6 -> 4.34 mm, vias 6 -> 0
- net Net-(D10-Pad1): track 4.86 -> 245.6 mm
- net Net-(D10-Pad2): track 243.3 -> 4.34 mm
- net Net-(D22-Pad2): track 211.8 -> 4.34 mm
- net Net-(D22-Pad1): track 4.86 -> 212.1 mm
- net Net-(D23-Pad1): track 4.86 -> 205.9 mm
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