File: pcb/kb-pcb.sch (KiCad schematic (older format))
At the start: 137 parts, among them U1 TEENSY2.0

Commit message: add solder points for pull-down resistors as in #3
Parts:
- added R1, R10, R11, R12, R13, R14, R2, R3, R4, R5, R6, R7, R8, R9: R, Resistors_Universal:Resistor_SMD+THTuniversal_0805to2512_RM10_HandSoldering, symbol R
Connections:
- net GND: now also R1.2, R10.2, R11.2, R12.2, R13.2, R14.2, R2.2, R3.2, R4.2, R5.2, R6.2, R8.2
- net at D14.2 (A), D28.2 (A), D42.2 (A)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: now also R14.1
- net at D10.2 (A), D24.2 (A), D38.2 (A)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: now also R10.1
- net at D23.2 (A), D37.2 (A), D51.2 (A)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: now also R9.1
- net at D22.2 (A), D36.2 (A), D50.2 (A)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: now also R8.1
- net at D1.2 (A), D15.2 (A), D29.2 (A)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: now also R1.1
- net at D16.2 (A), D2.2 (A), D30.2 (A)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: now also R2.1
- net at D17.2 (A), D3.2 (A), D31.2 (A)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: now also R3.1
- net at D18.2 (A), D32.2 (A), D4.2 (A)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: now also R4.1
- net at D19.2 (A), D33.2 (A), D47.2 (A)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: now also R5.1
- net at D20.2 (A), D34.2 (A), D48.2 (A)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: now also R6.1
- net at D13.2 (A), D27.2 (A), D41.2 (A)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: now also R13.1
- net at D12.2 (A), D26.2 (A), D40.2 (A)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: now also R12.1
- net at D11.2 (A), D25.2 (A), D39.2 (A)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: now also R11.1
- net at D21.2 (A), D35.2 (A), D49.2 (A)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: now also R7.1

Commit message: fix two unconnected resistors
Connections:
- net GND: now also R7.2, R9.2
Changed lines of the file:
@@
 EESchema Schematic File Version 2
-LIBS:power
-LIBS:device
-LIBS:transistors
-LIBS:conn
-LIBS:linear
-LIBS:regul
-LIBS:74xx
-LIBS:cmos4000
-LIBS:adc-dac
-LIBS:memory
-LIBS:xilinx
-LIBS:microcontrollers
-LIBS:dsp
-LIBS:microchip
-LIBS:analog_switches
-LIBS:motorola
-LIBS:texas
-LIBS:intel
-LIBS:audio
-LIBS:interface
-LIBS:digital-audio
-LIBS:philips
-LIBS:display
-LIBS:cypress
-LIBS:siliconi
-LIBS:opto
-LIBS:atmel
-LIBS:contrib
-LIBS:valves
 LIBS:components
 LIBS:cherry-mx-switch-revised
@@
 	1    0    0    -1
 $EndComp
+$Comp
+L R R13
+U 1 1 5A22289E
+P 20600 10950
+F 0 "R13" V 20680 10950 50  0000 C CNN
+F 1 "R" V 20600 10950 50  0000 C CNN
+F 2 "Resistors_Universal:Resistor_SMD+THTuniversal_0805to2512_RM10_HandSoldering" V 20530 10950 50  0001 C CNN
+F 3 "" H 20600 10950 50  0000 C CNN
+	1    20600 10950
+	1    0    0    -1
+$EndComp
+$Comp
+L R R14
+U 1 1 5A222CFE
+P 22100 10950
+F 0 "R14" V 22180 10950 50  0000 C CNN
+F 1 "R" V 22100 10950 50  0000 C CNN
+F 2 "Resistors_Universal:Resistor_SMD+THTuniversal_0805to2512_RM10_HandSoldering" V 22030 10950 50  0001 C CNN
+F 3 "" H 22100 10950 50  0000 C CNN
+	1    22100 10950
+	1    0    0    -1
+$EndComp
 Wire Wire Line
 	1300 6200 1300 5800
@@
 Wire Wire Line
 	10100 5250 10100 10800
-Wire Wire Line
-	900  11100 22100 11100
 Connection ~ 4100 11100
 Connection ~ 5600 11100
@@
 Wire Wire Line
 	900  3350 900  11100
-$Comp
-L R R13
-U 1 1 5A22289E
-P 20600 10950
-F 0 "R13" V 20680 10950 50  0000 C CNN
-F 1 "R" V 20600 10950 50  0000 C CNN
-F 2 "Resistors_Universal:Resistor_SMD+THTuniversal_0805to2512_RM10_HandSoldering" V 20530 10950 50  0001 C CNN
-F 3 "" H 20600 10950 50  0000 C CNN
-	1    20600 10950
-	1    0    0    -1
-$EndComp
-$Comp
-L R R14
-U 1 1 5A222CFE
-P 22100 10950
-F 0 "R14" V 22180 10950 50  0000 C CNN
-F 1 "R" V 22100 10950 50  0000 C CNN
-F 2 "Resistors_Universal:Resistor_SMD+THTuniversal_0805to2512_RM10_HandSoldering" V 22030 10950 50  0001 C CNN
-F 3 "" H 22100 10950 50  0000 C CNN
-	1    22100 10950
-	1    0    0    -1
-$EndComp
+Wire Wire Line
+	900  11100 22100 11100
+Wire Wire Line
+	11600 11100 11600 11100
+Connection ~ 11600 11100
+Wire Wire Line
+	14600 11100 14600 11100
+Connection ~ 14600 11100
 $EndSCHEMATC

Commit message: upgrade to Kicad 5 footprints
In doing so, I've updated the diodes to be N4148 diodes from the
official modules. Since those have slightly different footprints from
the original ones I used, I've modified the PCB layout accordingly.

I lost track of the original Teensy 2.0 footprint I created, so I'm
using a modified version of XenGi's footprint as well.
Parts:
- D1, D10, D11, D12, D13, D14, D15, D16, D17, D18, D19, D2, D20, D21, D22, D23, D24, D25, D26, D27, D28, D29, D3, D30, D31, D32, D33, D34, D35, D36, D37, D38, D39, D4, D40, D41, D42, D43, D44, D45, D46, D47, D48, D49, D5, D50, D51, D52, D53, D54, D55, D56, D57, D58, D59, D6, D60, D61, D62, D63, D64, D65, D66, D67, D68, D7, D8, D9: footprint modded_keyboard_components:diode -> Diode_THT:D_DO-35_SOD27_P7.62mm_Horizontal; symbol D -> kb-pcb-rescue:D
- R1, R10, R11, R12, R13, R14, R2, R3, R4, R5, R6, R7, R8, R9: symbol R -> kb-pcb-rescue:R
- S1, S10, S11, S12, S13, S14, S15, S16, S17, S18, S19, S2, S20, S21, S22, S23, S24, S25, S26, S27, S28, S29, S3, S30, S31, S32, S33, S34, S35, S36, S37, S38, S39, S4, S40, S41, S42, S43, S44, S45, S46, S47, S48, S49, S5, S50, S51, S52, S53, S54, S55, S56, S57, S58, S59, S6, S60, S61, S62, S63, S64, S65, S66, S67, S68, S7, S8, S9: symbol cherry-mx-switch-revised -> cherry-mx-switch-revised:cherry-mx-switch-revised
- U1: footprint modded_keyboard_components:TEENSY_2.0 -> teensy:Teensy2.0; symbol TEENSY2.0 -> components:TEENSY2.0
Connections:
- net at D4.1 (K): now also D18.1 (K), D32.1 (K), D46.1 (K), D60.1 (K), R4.1, U1.26 (PF4); no longer S4.1 (OUTPUT)
- net at D5.1 (K): now also D19.1 (K), D33.1 (K), D47.1 (K), D61.1 (K), R5.1, U1.27 (PF1); no longer S5.1 (OUTPUT)
- net at D6.1 (K): now also D20.1 (K), D34.1 (K), D48.1 (K), R6.1, U1.28 (PF0); no longer S6.1 (OUTPUT)
- net at D3.1 (K): now also D17.1 (K), D31.1 (K), D45.1 (K), D59.1 (K), R3.1, U1.25 (PF5); no longer S3.1 (OUTPUT)
- net at D2.1 (K): now also D16.1 (K), D30.1 (K), D44.1 (K), D58.1 (K), R2.1, U1.24 (PF6); no longer S2.1 (OUTPUT)
- net at D1.1 (K): now also D15.1 (K), D29.1 (K), D43.1 (K), D57.1 (K), R1.1, U1.23 (PF7); no longer S1.1 (OUTPUT)
- net at D7.1 (K): now also D21.1 (K), D35.1 (K), D49.1 (K), D62.1 (K), R7.1, U1.6 (PB7); no longer S7.1 (OUTPUT)
- net at D8.1 (K): now also D22.1 (K), D36.1 (K), D50.1 (K), D63.1 (K), R8.1, U1.22 (PB6); no longer S8.1 (OUTPUT)
- net at D9.1 (K): now also D23.1 (K), D37.1 (K), D51.1 (K), R9.1, U1.21 (PB5); no longer S9.1 (OUTPUT)
- net at D10.1 (K): now also D24.1 (K), D38.1 (K), D52.1 (K), D64.1 (K), R10.1, U1.20 (PB4); no longer S10.1 (OUTPUT)
- net at D11.1 (K): now also D25.1 (K), D39.1 (K), D53.1 (K), D65.1 (K), R11.1, U1.5 (PB3); no longer S11.1 (OUTPUT)
- net at D12.1 (K): now also D26.1 (K), D40.1 (K), D54.1 (K), D66.1 (K), R12.1, U1.4 (PB2); no longer S12.1 (OUTPUT)
- net at D13.1 (K): now also D27.1 (K), D41.1 (K), D55.1 (K), D67.1 (K), R13.1, U1.3 (PB1); no longer S13.1 (OUTPUT)
- net at D14.1 (K): now also D28.1 (K), D42.1 (K), D56.1 (K), D68.1 (K), R14.1, U1.2 (PB0); no longer S14.1 (OUTPUT)
- net at S18.1 (OUTPUT): now also D18.2 (A); no longer D18.1 (K)
- net at S19.1 (OUTPUT): now also D19.2 (A); no longer D19.1 (K)
- net at S20.1 (OUTPUT): now also D20.2 (A); no longer D20.1 (K)
- net at S17.1 (OUTPUT): now also D17.2 (A); no longer D17.1 (K)
- net at S16.1 (OUTPUT): now also D16.2 (A); no longer D16.1 (K)
- net at S15.1 (OUTPUT): now also D15.2 (A); no longer D15.1 (K)
- net at S21.1 (OUTPUT): now also D21.2 (A); no longer D21.1 (K)
- net at S22.1 (OUTPUT): now also D22.2 (A); no longer D22.1 (K)
- net at S23.1 (OUTPUT): now also D23.2 (A); no longer D23.1 (K)
- net at S24.1 (OUTPUT): now also D24.2 (A); no longer D24.1 (K)
- net at S25.1 (OUTPUT): now also D25.2 (A); no longer D25.1 (K)
- net at S26.1 (OUTPUT): now also D26.2 (A); no longer D26.1 (K)
- net at S27.1 (OUTPUT): now also D27.2 (A); no longer D27.1 (K)
- net at S28.1 (OUTPUT): now also D28.2 (A); no longer D28.1 (K)
- net at S32.1 (OUTPUT): now also D32.2 (A); no longer D32.1 (K)
- net at S33.1 (OUTPUT): now also D33.2 (A); no longer D33.1 (K)
- net at S34.1 (OUTPUT): now also D34.2 (A); no longer D34.1 (K)
- net at S31.1 (OUTPUT): now also D31.2 (A); no longer D31.1 (K)
- net at S30.1 (OUTPUT): now also D30.2 (A); no longer D30.1 (K)
- net at S29.1 (OUTPUT): now also D29.2 (A); no longer D29.1 (K)
- net at S35.1 (OUTPUT): now also D35.2 (A); no longer D35.1 (K)
- net at S36.1 (OUTPUT): now also D36.2 (A); no longer D36.1 (K)
- net at S37.1 (OUTPUT): now also D37.2 (A); no longer D37.1 (K)
- net at S38.1 (OUTPUT): now also D38.2 (A); no longer D38.1 (K)
- net at S39.1 (OUTPUT): now also D39.2 (A); no longer D39.1 (K)
- net at S40.1 (OUTPUT): now also D40.2 (A); no longer D40.1 (K)
- net at S41.1 (OUTPUT): now also D41.2 (A); no longer D41.1 (K)
- net at S42.1 (OUTPUT): now also D42.2 (A); no longer D42.1 (K)
- net at S46.1 (OUTPUT): now also D46.2 (A); no longer D46.1 (K)
- net at S47.1 (OUTPUT): now also D47.2 (A); no longer D47.1 (K)
- net at S48.1 (OUTPUT): now also D48.2 (A); no longer D48.1 (K)
- net at S45.1 (OUTPUT): now also D45.2 (A); no longer D45.1 (K)
- net at S44.1 (OUTPUT): now also D44.2 (A); no longer D44.1 (K)
- net at S43.1 (OUTPUT): now also D43.2 (A); no longer D43.1 (K)
- net at S49.1 (OUTPUT): now also D49.2 (A); no longer D49.1 (K)
- net at S50.1 (OUTPUT): now also D50.2 (A); no longer D50.1 (K)
- net at S51.1 (OUTPUT): now also D51.2 (A); no longer D51.1 (K)
- net at S52.1 (OUTPUT): now also D52.2 (A); no longer D52.1 (K)
- net at S53.1 (OUTPUT): now also D53.2 (A); no longer D53.1 (K)
- net at S54.1 (OUTPUT): now also D54.2 (A); no longer D54.1 (K)
- net at S55.1 (OUTPUT): now also D55.2 (A); no longer D55.1 (K)
- net at S56.1 (OUTPUT): now also D56.2 (A); no longer D56.1 (K)
- net at S60.1 (OUTPUT): now also D60.2 (A); no longer D60.1 (K)
- net at S61.1 (OUTPUT): now also D61.2 (A); no longer D61.1 (K)
- net at S59.1 (OUTPUT): now also D59.2 (A); no longer D59.1 (K)
- net at S58.1 (OUTPUT): now also D58.2 (A); no longer D58.1 (K)
- net at S57.1 (OUTPUT): now also D57.2 (A); no longer D57.1 (K)
- net at S62.1 (OUTPUT): now also D62.2 (A); no longer D62.1 (K)
- net at S63.1 (OUTPUT): now also D63.2 (A); no longer D63.1 (K)
- net at S64.1 (OUTPUT): now also D64.2 (A); no longer D64.1 (K)
- net at S65.1 (OUTPUT): now also D65.2 (A); no longer D65.1 (K)
- net at S66.1 (OUTPUT): now also D66.2 (A); no longer D66.1 (K)
- net at S67.1 (OUTPUT): now also D67.2 (A); no longer D67.1 (K)
- net at S68.1 (OUTPUT): now also D68.2 (A); no longer D68.1 (K)
- new net: D4.2 (A), S4.1 (OUTPUT)
- new net: D5.2 (A), S5.1 (OUTPUT)
- new net: D6.2 (A), S6.1 (OUTPUT)
- new net: D3.2 (A), S3.1 (OUTPUT)
- new net: D2.2 (A), S2.1 (OUTPUT)
- new net: D1.2 (A), S1.1 (OUTPUT)
- new net: D7.2 (A), S7.1 (OUTPUT)
- new net: D8.2 (A), S8.1 (OUTPUT)
- new net: D9.2 (A), S9.1 (OUTPUT)
- new net: D10.2 (A), S10.1 (OUTPUT)
- new net: D11.2 (A), S11.1 (OUTPUT)
- new net: D12.2 (A), S12.1 (OUTPUT)
- new net: D13.2 (A), S13.1 (OUTPUT)
- new net: D14.2 (A), S14.1 (OUTPUT)
